Commit message: modify feed forwrod torque computation

File: resources/robots/hex_magnetic/urdf/hex_all.urdf (robot description, URDF)
Before this commit: robot hex_magnetic, 43 links, 42 joints
Links:
- removed link l_lb_suck_pitch
- removed link l_lb_suck_roll
- removed link l_lf_suck_pitch
- removed link l_lf_suck_roll
- removed link l_lm_suck_pitch
- removed link l_lm_suck_roll
- removed link l_rb_suck_pitch
- removed link l_rb_suck_roll
- removed link l_rf_suck_pitch
- removed link l_rf_suck_roll
- removed link l_rm_suck_pitch
- removed link l_rm_suck_roll
- added link l_lb_ball1, mass 0.001; visual sphere radius=0.008
- added link l_lb_ball2, mass 0.001; visual sphere radius=0.008
- added link l_lb_empty
- added link l_lb_toe, mass 1e-2; collision cylinder length=0.008 radius=0.018; visual cylinder length=0.008 radius=0.018
- added link l_lf_ball1, mass 0.001; visual sphere radius=0.008
- added link l_lf_ball2, mass 0.001; visual sphere radius=0.008
- added link l_lf_empty
- added link l_lf_toe, mass 1e-2; collision cylinder length=0.008 radius=0.018; visual cylinder length=0.008 radius=0.018
- added link l_lm_ball1, mass 0.001; visual sphere radius=0.008
- added link l_lm_ball2, mass 0.001; visual sphere radius=0.008
- added link l_lm_empty
- added link l_lm_toe, mass 1e-2; collision cylinder length=0.008 radius=0.018; visual cylinder length=0.008 radius=0.018
- added link l_rb_ball1, mass 0.001; visual sphere radius=0.008
- added link l_rb_ball2, mass 0.001; visual sphere radius=0.008
- added link l_rb_empty
- added link l_rb_toe, mass 1e-2; collision cylinder length=0.008 radius=0.018; visual cylinder length=0.008 radius=0.018
- added link l_rf_ball1, mass 0.001; visual sphere radius=0.008
- added link l_rf_ball2, mass 0.001; visual sphere radius=0.008
- added link l_rf_empty
- added link l_rf_toe, mass 1e-2; collision cylinder length=0.008 radius=0.018; visual cylinder length=0.008 radius=0.018
- added link l_rm_ball1, mass 0.001; visual sphere radius=0.008
- added link l_rm_ball2, mass 0.001; visual sphere radius=0.008
- added link l_rm_empty
- added link l_rm_toe, mass 1e-2; collision cylinder length=0.008 radius=0.018; visual cylinder length=0.008 radius=0.018
- link l_lb_ankle: geometry collision sphere radius=0.0265; visual mesh filename=../course_meshes/l_lf_ankle.STL
- link l_lb_suck: geometry collision cylinder length=0.012 radius=0.02; visual mesh filename=../course_meshes/l_lf_suck.STL
- link l_lb_thigh: geometry collision sphere radius=0.0265; visual mesh filename=../course_meshes/l_lf_thigh.STL
- link l_lf_ankle: geometry collision sphere radius=0.0265; visual mesh filename=../course_meshes/l_lf_ankle.STL
- link l_lf_suck: geometry collision cylinder length=0.012 radius=0.02; visual mesh filename=../course_meshes/l_lf_suck.STL
- link l_lf_thigh: geometry collision sphere radius=0.0265; visual mesh filename=../course_meshes/l_lf_thigh.STL
- link l_lm_ankle: geometry collision sphere radius=0.0265; visual mesh filename=../course_meshes/l_lf_ankle.STL
- link l_lm_suck: geometry collision cylinder length=0.012 radius=0.02; visual mesh filename=../course_meshes/l_lf_suck.STL
- link l_lm_thigh: geometry collision sphere radius=0.0265; visual mesh filename=../course_meshes/l_lf_thigh.STL
- link l_rb_ankle: geometry collision sphere radius=0.0265; visual mesh filename=../course_meshes/l_rf_ankle.STL
- link l_rb_suck: geometry collision cylinder length=0.012 radius=0.02; visual mesh filename=../course_meshes/l_rf_suck.STL
- link l_rb_thigh: geometry collision sphere radius=0.0265; visual mesh filename=../course_meshes/l_rf_thigh.STL
- link l_rf_ankle: geometry collision sphere radius=0.0265; visual mesh filename=../course_meshes/l_rf_ankle.STL
- link l_rf_suck: geometry collision cylinder length=0.012 radius=0.02; visual mesh filename=../course_meshes/l_rf_suck.STL
- link l_rf_thigh: geometry collision sphere radius=0.0265; visual mesh filename=../course_meshes/l_rf_thigh.STL
- link l_rm_ankle: geometry collision sphere radius=0.0265; visual mesh filename=../course_meshes/l_rf_ankle.STL
- link l_rm_suck: geometry collision cylinder length=0.012 radius=0.02; visual mesh filename=../course_meshes/l_rf_suck.STL
- link l_rm_thigh: geometry collision sphere radius=0.0265; visual mesh filename=../course_meshes/l_rf_thigh.STL
Joints:
- removed joint j_lb_suck_pitch
- removed joint j_lb_suck_roll
- removed joint j_lf_suck_pitch
- removed joint j_lf_suck_roll
- removed joint j_lm_suck_pitch
- removed joint j_lm_suck_roll
- removed joint j_rb_suck_pitch
- removed joint j_rb_suck_roll
- removed joint j_rf_suck_pitch
- removed joint j_rf_suck_roll
- removed joint j_rm_suck_pitch
- removed joint j_rm_suck_roll
- added joint j_lb_ball1: type revolute, parent l_lb_foot, child l_lb_ball1, origin xyz=0.001 0 0 rpy=0 1.5707963267949 0, axis 1 0 0, limit lower=-0.3490658503988659 upper=0.3490658503988659 effort=0.2 velocity=2
- added joint j_lb_ball2: type revolute, parent l_lb_ball1, child l_lb_ball2, origin xyz=0 0 0 rpy=0 0 0, axis 0 1 0, limit lower=-0.3490658503988659 upper=0.3490658503988659 effort=0.2 velocity=2
- added joint j_lb_empty: type fixed, parent l_lb_toe, child l_lb_empty, origin xyz=0 0 0 rpy=0 0 0
- added joint j_lb_toe: type fixed, parent l_lb_suck, child l_lb_toe, origin xyz=0 0 0.026 rpy=0 0 0
- added joint j_lf_ball1: type revolute, parent l_lf_foot, child l_lf_ball1, origin xyz=0.001 0 0 rpy=0 1.5707963267949 0, axis 1 0 0, limit lower=-0.3490658503988659 upper=0.3490658503988659 effort=0.2 velocity=2
- added joint j_lf_ball2: type revolute, parent l_lf_ball1, child l_lf_ball2, origin xyz=0 0 0 rpy=0 0 0, axis 0 1 0, limit lower=-0.3490658503988659 upper=0.3490658503988659 effort=0.2 velocity=2
- added joint j_lf_empty: type fixed, parent l_lf_toe, child l_lf_empty, origin xyz=0 0 0 rpy=0 0 0
- added joint j_lf_toe: type fixed, parent l_lf_suck, child l_lf_toe, origin xyz=0 0 0.026 rpy=0 0 0
- added joint j_lm_ball1: type revolute, parent l_lm_foot, child l_lm_ball1, origin xyz=0.001 0 0 rpy=0 1.5707963267949 0, axis 1 0 0, limit lower=-0.3490658503988659 upper=0.3490658503988659 effort=0.2 velocity=2
- added joint j_lm_ball2: type revolute, parent l_lm_ball1, child l_lm_ball2, origin xyz=0 0 0 rpy=0 0 0, axis 0 1 0, limit lower=-0.3490658503988659 upper=0.3490658503988659 effort=0.2 velocity=2
- added joint j_lm_empty: type fixed, parent l_lm_toe, child l_lm_empty, origin xyz=0 0 0 rpy=0 0 0
- added joint j_lm_toe: type fixed, parent l_lm_suck, child l_lm_toe, origin xyz=0 0 0.026 rpy=0 0 0
- added joint j_rb_ball1: type revolute, parent l_rb_foot, child l_rb_ball1, origin xyz=0.001 0 0 rpy=0 1.5707963267949 0, axis 1 0 0, limit lower=-0.3490658503988659 upper=0.3490658503988659 effort=0.2 velocity=2
- added joint j_rb_ball2: type revolute, parent l_rb_ball1, child l_rb_ball2, origin xyz=0 0 0 rpy=0 0 0, axis 0 1 0, limit lower=-0.3490658503988659 upper=0.3490658503988659 effort=0.2 velocity=2
- added joint j_rb_empty: type fixed, parent l_rb_toe, child l_rb_empty, origin xyz=0 0 0 rpy=0 0 0
- added joint j_rb_toe: type fixed, parent l_rb_suck, child l_rb_toe, origin xyz=0 0 0.026 rpy=0 0 0
- added joint j_rf_ball1: type revolute, parent l_rf_foot, child l_rf_ball1, origin xyz=0.001 0 0 rpy=0 1.5707963267949 0, axis 1 0 0, limit lower=-0.3490658503988659 upper=0.3490658503988659 effort=0.2 velocity=2
- added joint j_rf_ball2: type revolute, parent l_rf_ball1, child l_rf_ball2, origin xyz=0 0 0 rpy=0 0 0, axis 0 1 0, limit lower=-0.3490658503988659 upper=0.3490658503988659 effort=0.2 velocity=2
- added joint j_rf_empty: type fixed, parent l_rf_toe, child l_rf_empty, origin xyz=0 0 0 rpy=0 0 0
- added joint j_rf_toe: type fixed, parent l_rf_suck, child l_rf_toe, origin xyz=0 0 0.026 rpy=0 0 0
- added joint j_rm_ball1: type revolute, parent l_rm_foot, child l_rm_ball1, origin xyz=0.001 0 0 rpy=0 1.5707963267949 0, axis 1 0 0, limit lower=-0.3490658503988659 upper=0.3490658503988659 effort=0.2 velocity=2
- added joint j_rm_ball2: type revolute, parent l_rm_ball1, child l_rm_ball2, origin xyz=0 0 0 rpy=0 0 0, axis 0 1 0, limit lower=-0.3490658503988659 upper=0.3490658503988659 effort=0.2 velocity=2
- added joint j_rm_empty: type fixed, parent l_rm_toe, child l_rm_empty, origin xyz=0 0 0 rpy=0 0 0
- added joint j_rm_toe: type fixed, parent l_rm_suck, child l_rm_toe, origin xyz=0 0 0.026 rpy=0 0 0
- joint j_lb_suck: parent l_lb_suck_pitch -> l_lb_ball2
- joint j_lf_suck: parent l_lf_suck_pitch -> l_lf_ball2
- joint j_lm_suck: parent l_lm_suck_pitch -> l_lm_ball2
- joint j_rb_suck: parent l_rb_suck_pitch -> l_rb_ball2
- joint j_rf_suck: parent l_rf_suck_pitch -> l_rf_ball2
- joint j_rm_suck: parent l_rm_suck_pitch -> l_rm_ball2

File: resources/robots/hex_magnetic/urdf/hex_all_magnetic.xacro (robot description, xacro)
@@ -7,5 +7,5 @@
       <origin xyz="-0.00031149 -7.4441E-05 0.0027279" rpy="0 0 0" />
       <mass value="6.023" />
-      <inertia ixx="0.169108146" ixy="-0.000168229" ixz="0.000016567" iyy="0.040037856" iyz="-0.001521188" izz="0.2016899" />
+      <inertia ixx="0.169108146" ixy="-0.000168229" ixz="0.000016567" iyy="0.0260037856" iyz="-0.001521188" izz="0.2016899" />
     </inertial>
     <visual>
@@ -50,5 +50,5 @@
         <origin xyz="0.072 0 0" rpy="0 0 0"/>
         <geometry>
-          <sphere radius="0.045"/>
+          <sphere radius="0.0265"/>
         </geometry>
       </collision>
@@ -87,5 +87,5 @@
         <origin xyz="0.065 0 0" rpy="0 0 0" />
         <geometry>
-          <box size="0.06 0.04 0.08" />
+          <box size="0.06 0.026 0.08" />
         </geometry>
       </collision> -->
@@ -122,5 +122,5 @@
         <origin xyz="0 0 0" rpy="0 0 0"/>
         <geometry>
-          <sphere radius="0.045"/>
+          <sphere radius="0.0265"/>
         </geometry>
       </collision>
@@ -162,5 +162,5 @@
       <limit lower="${-pi/2.0}" upper="${pi/2.0}" effort="0.45" velocity="${pi}" />
     </joint>
-    <link name="l_${prefix}_suck_roll">
+    <link name="l_${prefix}_ball1">
       <inertial>
         <origin xyz="0 0 0" rpy="0 0 0" />
@@ -178,12 +178,12 @@
       </visual>
     </link>
-    <joint name="j_${prefix}_suck_roll" type="revolute">
+    <joint name="j_${prefix}_ball1" type="revolute">
       <origin xyz="0.001 0 0" rpy="0 1.5707963267949 0" />
       <parent link="l_${prefix}_foot" />
-      <child link="l_${prefix}_suck_roll" />
+      <child link="l_${prefix}_ball1" />
       <axis xyz="1 0 0" />
       <limit lower="${-pi/9.0}" upper="${pi/9.0}" effort="0.2" velocity="2" />
     </joint>
-    <link name="l_${prefix}_suck_pitch">
+    <link name="l_${prefix}_ball2">
       <inertial>
         <origin xyz="0 0 0" rpy="0 0 0" />
@@ -201,8 +201,8 @@
       </visual>
     </link>
-    <joint name="j_${prefix}_suck_pitch" type="revolute">
+    <joint name="j_${prefix}_ball2" type="revolute">
       <origin xyz="0 0 0" rpy="0 0 0" />
-      <parent link="l_${prefix}_suck_roll" />
-      <child link="l_${prefix}_suck_pitch" />
+      <parent link="l_${prefix}_ball1" />
+      <child link="l_${prefix}_ball2" />
       <axis xyz="0 1 0" />
       <limit lower="${-pi/9.0}" upper="${pi/9.0}" effort="0.2" velocity="2" />
@@ -224,7 +224,7 @@
       </visual>
       <collision>
-        <origin xyz="0 0 0.02" rpy="0 0 0" />
-        <geometry>
-          <cylinder length="0.02" radius="0.02" />
+        <origin xyz="0 0 0.014" rpy="0 0 0" />
+        <geometry>
+          <cylinder length="0.012" radius="0.02" />
         </geometry>
       </collision>
@@ -232,8 +232,36 @@
     <joint name="j_${prefix}_suck" type="revolute">
       <origin xyz="0 0 0" rpy="0 0 0" />
-      <parent link="l_${prefix}_suck_pitch" />
+      <parent link="l_${prefix}_ball2" />
       <child link="l_${prefix}_suck" />
       <axis xyz="0 0 1" />
       <limit lower="${-pi}" upper="${pi}" effort="0.5" velocity="5" />
+    </joint>
+      <!-- 添加toe是为了检测吸附面是否接触碰撞 避免电磁铁侧面碰撞也误认为是吸附面接触 toe比suck小一点 且只有在suck底面露出来一点 -->
+    <link name="l_${prefix}_toe">
+      <inertial>
+        <origin xyz="0 0 0" rpy="0 0 0" />
+        <mass value="1e-2"/>
+        <inertia ixx="1.053e-6" ixy="0" ixz="0" iyy="1.053e-6" iyz="0" izz="2.0e-6" />
+      </inertial>
+      <visual>
+        <origin xyz="0 0 0" rpy="0 0 0" />
+        <geometry> <cylinder radius="0.018" length="0.008" /> </geometry>
+      </visual>
+      <collision>
+        <origin xyz="0 0 0" rpy="0 0 0" />
+        <geometry> <cylinder radius="0.018" length="0.008" /> </geometry>
+      </collision>
+    </link>
+    <joint name="j_${prefix}_toe" type="fixed">
+      <origin xyz="0 0 0.026" rpy="0 0 0"/>
+      <parent link="l_${prefix}_suck"/>
+      <child link="l_${prefix}_toe"/>
+    </joint>
+    <!-- 添加 empty 是为了方便吸附力的施加 给suck toe  empy三个位置按照圆心分别设置三个正向力 能更好的模拟吸盘对额外力和扭矩的反应-->
+    <link name="l_${prefix}_empty"/>
+    <joint name="j_${prefix}_empty" type="fixed">
+      <origin xyz="0 0 0" rpy="0 0 0"/>
+      <parent link="l_${prefix}_toe"/>
+      <child link="l_${prefix}_empty"/>
     </joint>
   </xacro:macro>
@@ -263,5 +291,5 @@
         <origin xyz="0.072 0 0" rpy="0 0 0"/>
         <geometry>
-          <sphere radius="0.045"/>
+          <sphere radius="0.0265"/>
         </geometry>
       </collision>
@@ -300,5 +328,5 @@
         <origin xyz="0.065 0 0" rpy="0 0 0" />
         <geometry>
-          <box size="0.06 0.04 0.08" />
+          <box size="0.06 0.026 0.08" />
         </geometry>
       </collision> -->
@@ -335,5 +363,5 @@
         <origin xyz="0 0 0" rpy="0 0 0"/>
         <geometry>
-          <sphere radius="0.045"/>
+          <sphere radius="0.0265"/>
         </geometry>
       </collision>
@@ -369,5 +397,5 @@
       <limit lower="${-pi/2.0}" upper="${pi/2.0}" effort="0.45" velocity="${pi}" />
     </joint>
-    <link name="l_${prefix}_suck_roll">
+    <link name="l_${prefix}_ball1">
       <inertial>
         <origin xyz="0 0 0" rpy="0 0 0" />
@@ -385,12 +413,12 @@
       </visual>
     </link>
-    <joint name="j_${prefix}_suck_roll" type="revolute">
+    <joint name="j_${prefix}_ball1" type="revolute">
       <origin xyz="0.001 0 0" rpy="0 1.5707963267949 0" />
       <parent link="l_${prefix}_foot" />
-      <child link="l_${prefix}_suck_roll" />
+      <child link="l_${prefix}_ball1" />
       <axis xyz="1 0 0" />
       <limit lower="${-pi/9.0}" upper="${pi/9.0}" effort="0.2" velocity="2" />
     </joint>
-    <link name="l_${prefix}_suck_pitch">
+    <link name="l_${prefix}_ball2">
       <inertial>
         <origin xyz="0 0 0" rpy="0 0 0" />
@@ -408,8 +436,8 @@
       </visual>
     </link>
-    <joint name="j_${prefix}_suck_pitch" type="revolute">
+    <joint name="j_${prefix}_ball2" type="revolute">
       <origin xyz="0 0 0" rpy="0 0 0" />
-      <parent link="l_${prefix}_suck_roll" />
-      <child link="l_${prefix}_suck_pitch" />
+      <parent link="l_${prefix}_ball1" />
+      <child link="l_${prefix}_ball2" />
       <axis xyz="0 1 0" />
       <limit lower="${-pi/9.0}" upper="${pi/9.0}" effort="0.2" velocity="2" />
@@ -431,7 +459,7 @@
       </visual>
       <collision>
-        <origin xyz="0 0 0.02" rpy="0 0 0" />
-        <geometry>
-          <cylinder length="0.02" radius="0.02" />
+        <origin xyz="0 0 0.014" rpy="0 0 0" />
+        <geometry>
+          <cylinder length="0.012" radius="0.02" />
         </geometry>
       </collision>
@@ -439,8 +467,36 @@
     <joint name="j_${prefix}_suck" type="revolute">
       <origin xyz="0 0 0" rpy="0 0 0" />
-      <parent link="l_${prefix}_suck_pitch" />
+      <parent link="l_${prefix}_ball2" />
       <child link="l_${prefix}_suck" />
       <axis xyz="0 0 1" />
       <limit lower="${-pi}" upper="${pi}" effort="0.5" velocity="5" />
+    </joint>
+      <!-- 添加toe是为了检测吸附面是否接触碰撞 避免电磁铁侧面碰撞也误认为是吸附面接触 toe比suck小一点 且只有在suck底面露出来一点 -->
+    <link name="l_${prefix}_toe">
+      <inertial>
+        <origin xyz="0 0 0" rpy="0 0 0" />
+        <mass value="1e-2"/>
+        <inertia ixx="1.053e-6" ixy="0" ixz="0" iyy="1.053e-6" iyz="0" izz="2.0e-6" />
+      </inertial>
+      <visual>
+        <origin xyz="0 0 0" rpy="0 0 0" />
+        <geometry> <cylinder radius="0.018" length="0.008" /> </geometry>
+      </visual>
+      <collision>
+        <origin xyz="0 0 0" rpy="0 0 0" />
+        <geometry> <cylinder radius="0.018" length="0.008" /> </geometry>
+      </collision>
+    </link>
+    <joint name="j_${prefix}_toe" type="fixed">
+      <origin xyz="0 0 0.026" rpy="0 0 0"/>
+      <parent link="l_${prefix}_suck"/>
+      <child link="l_${prefix}_toe"/>
+    </joint>
+    <!-- 添加 empty 是为了方便吸附力的施加 给suck toe  empy三个位置按照圆心分别设置三个正向力 能更好的模拟吸盘对额外力和扭矩的反应-->
+    <link name="l_${prefix}_empty"/>
+    <joint name="j_${prefix}_empty" type="fixed">
+      <origin xyz="0 0 0" rpy="0 0 0"/>
+      <parent link="l_${prefix}_toe"/>
+      <child link="l_${prefix}_empty"/>
     </joint>
   </xacro:macro>
